File: Electronics/KiCAD/EMGsensor_v2.1/EMGsensor_v2.1.sch (KiCad schematic (older format))
At the start: 37 parts, among them J1 Conn_01x03_Male, J2 Conn_01x02_Male, J3 Conn_01x03_Male, J4 SHIFT, J5 NO_SHIFT, U1 OPA4234P, U2 AD623, U3 OPA4234P

Commit message: Create PCB board
Parts:
- renumbered U3 to U1
Connections:
- net at R3.1: now also J3.3 (Pin_3); no longer J3.1 (Pin_1)
- net at R4.1: now also J3.1 (Pin_1); no longer J3.3 (Pin_3)
- no-connect marks 2 -> 1
Other:
- moved on the sheet: C1, C10, C11, C12, C2, C3, C4, C5, C6, C7, C8, C9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
