File: Electronics/KiCAD/EMGsensor_v2.1/_autosave-EMGsensor_v2.1.kicad_pcb (KiCad board)
At the start: 2 copper layers, 36 parts, among them J1 Conn_01x03_Male, J2 Conn_01x02_Male, J3 Conn_01x03_Male, J4 SHIFT, J5 NO_SHIFT, U1 OPA4234P, U2 AD623

Commit message: Create PCB board
Parts:
- moved J1 102.4 mm to (71.1, 118.1)
- moved J3 102.3 mm to (65.4, 107.3), turned to 90 degrees
- moved C5 90.7 mm to (85.7, 102.3), turned to 270 degrees
- moved C3 85.1 mm to (80.6, 98.5), turned to 270 degrees
- moved R3 79.1 mm to (67.9, 98.4)
- moved C4 74.4 mm to (80.6, 106.1), turned to 270 degrees
- moved R5 63.8 mm to (90.8, 97.2)
- moved C1 58.4 mm to (120.0, 94.0), turned to 90 degrees
- moved U1 55.7 mm to (130.2, 92.7)
- moved J2 52.2 mm to (84.5, 118.1), turned to 180 degrees
- moved R15 51.8 mm to (164.5, 84.5)
- moved U2 51.4 mm to (90.8, 102.2)
- moved R6 51.0 mm to (111.1, 107.3), turned to 270 degrees
- moved R1 49.8 mm to (106.0, 94.0)
- moved C6 49.7 mm to (126.4, 99.7), turned to 270 degrees
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Connections:
- R3 pad 1: Net-(J3-Pad1) -> Net-(J3-Pad3)
- R4 pad 1: Net-(J3-Pad3) -> Net-(J3-Pad1)
